File: hardware/Cx56-12xxx-serial-adapter/Cx56-12xxx-serial-adapter.kicad_pcb (KiCad board)
At the start: 2 copper layers, 70 x 23 mm, 14 parts, among them J1 Conn_01x05_Pin, U1 74HC595, U2 74HC595, U3 CC56-12EWA

Commit message: 002: from MSB to LSB shift register data transmission
Parts:
- moved C1 91.4 mm to (96.2, 70.9)
- moved C2 91.4 mm to (128.0, 70.9)
- moved J1 91.4 mm to (78.2, 70.1)
- moved R1 91.4 mm to (106.9, 61.6)
- moved R3 91.4 mm to (112.0, 68.5)
- moved R4 91.4 mm to (106.9, 68.5)
- moved R5 91.4 mm to (104.4, 68.5)
- moved U3 91.4 mm to (104.4, 72.5)
- moved R2 91.4 mm to (117.1, 61.6)
- moved R6 91.4 mm to (109.5, 61.6)
- moved R7 91.4 mm to (114.5, 68.5)
- moved R8 91.4 mm to (109.5, 68.5)
- moved U1 91.4 mm to (94.8, 63.7)
- moved U2 91.4 mm to (126.6, 63.7)
Connections:
- J1 pad 2: SRCLK/SHC -> VCC
- J1 pad 3: RCLK/STC -> SRCLK/SHC
- J1 pad 4: SER/DS -> RCLK/STC
- J1 pad 5: VCC -> SER/DS
- U1 pad 1: g' -> b'
- U1 pad 15: dp' -> a'
- U1 pad 2: f' -> c'
- U1 pad 3: e' -> d'
- U1 pad 4: d' -> e'
- U1 pad 5: c' -> f'
- U1 pad 6: b' -> g'
- U1 pad 7: a' -> dp'
- U2 pad 1: unconnected-(U2-QB-Pad1) -> D3
- U2 pad 15: unconnected-(U2-QA-Pad15) -> D4
- U2 pad 2: unconnected-(U2-QC-Pad2) -> D2
- U2 pad 3: unconnected-(U2-QD-Pad3) -> D1
- U2 pad 4: D1 -> unconnected-(U2-QE-Pad4)
- U2 pad 5: D2 -> unconnected-(U2-QF-Pad5)
- U2 pad 6: D3 -> unconnected-(U2-QG-Pad6)
- U2 pad 7: D4 -> unconnected-(U2-QH-Pad7)
Routing:
- net SRCLK/SHC: track 77.0 -> 48.6 mm, vias 1 -> 3
- net RCLK/STC: track 77.4 -> 49.8 mm, vias 1 -> 3
- net D3: track 36.9 -> 16.8 mm
- net MSB-LSB: track 54.2 -> 43.6 mm
- net VCC: track 94.1 -> 104.0 mm, vias 6 -> 2
- net D2: track 33.1 -> 23.7 mm, vias 2 -> 0
- net dp': track 21.4 -> 13.0 mm, vias 0 -> 2
- net a': track 12.1 -> 16.1 mm
- net c': track 16.9 -> 20.6 mm
- net g': track 21.5 -> 18.7 mm, vias 0 -> 2
- net GND: track 85.3 -> 87.5 mm, vias 4 -> 0
- net b': track 23.0 -> 21.2 mm
- net e': track 9.46 -> 10.9 mm
- net d': track 12.0 -> 13.4 mm, vias 2 -> 0
- net f': track 14.5 -> 13.1 mm, vias 0 -> 2
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Other:
- board text added: "Author: Maksym Palii Date: 23-Mar-2024 Revision: 2.0"
- board text added: "Cx56-12xxx serial adapter"
- board text added: "D1"
- board text added: "D2"
- board text added: "D3"
- board text added: "D4"
- board text added: "GND"
- board text added: "RCLK/STC"
- board text added: "SER/DS"
- board text added: "SRCLK/SHC"
- board text added: "VCC"
- board text added: "a"
- board text added: "b"
- board text added: "c"
- board text added: "d"
- board text added: "dp"
- board text added: "e"
- board text added: "f"
- board text added: "g"
